Commit message: up

File: bt6/ros2_ws/src/my_robot_description/urdf/my_robot.urdf.xacro (robot description, xacro)
@@ -1,203 +1,9 @@
 <?xml version="1.0"?>
 <robot xmlns:xacro="http://www.ros.org/wiki/xacro" name="my_robot">
-    <xacro:property name="base_width" value="0.4"/>
-    <xacro:property name="base_length" value="0.6"/>
-    <xacro:property name="base_height" value="0.2"/>
-    <xacro:property name="wheel_radius" value="0.1"/>
-    <xacro:property name="wheel_width" value="0.05"/>
-    <xacro:property name="wheel_ygap" value="0.025"/>
-    <xacro:property name="wheel_zoff" value="0.05"/>
-    <xacro:property name="wheel_xoff" value="0.15"/>
-    <xacro:property name="caster_xoff" value="0.2"/>
-    <!-- Define intertial macros -->
-    <xacro:macro name="box_inertia" params="m w h d">
-        <inertial>
-            <origin xyz="0 0 0" rpy="${pi/2} 0 ${pi/2}"/>
-            <mass value="${m}"/>
-            <inertia ixx="${(m/12) * (h*h + d*d)}" ixy="0.0" ixz="0.0" iyy="${(m/12) * (w*w + d*d)}" iyz="0.0" izz="${(m/12) * (w*w + h*h)}"/>
-        </inertial>
-    </xacro:macro>
-    <xacro:macro name="cylinder_inertia" params="m r h">
-        <inertial>
-            <origin xyz="0 0 0" rpy="${pi/2} 0 0" />
-            <mass value="${m}"/>
-            <inertia ixx="${(m/12) * (3*r*r + h*h)}" ixy = "0" ixz = "0" iyy="${(m/12) * (3*r*r + h*h)}" iyz = "0" izz="${(m/2) * (r*r)}"/>
-        </inertial>
-    </xacro:macro>
-    <xacro:macro name="sphere_inertia" params="m r">
-        <inertial>
-            <mass value="${m}"/>
-            <inertia ixx="${(2/5) * m * (r*r)}" ixy="0.0" ixz="0.0" iyy="${(2/5) * m * (r*r)}" iyz="0.0" izz="${(2/5) * m * (r*r)}"/>
-        </inertial>
-    </xacro:macro>
-    <!-- Robot Body -->
-    <link name="base_footprint"/>
-    <joint name="base_joint" type="fixed">
-        <parent link="base_footprint"/>
-        <child link="base_link"/>
-        <origin xyz="0.0 0.0 ${wheel_radius+wheel_zoff}" rpy="0 0 0"/>
-    </joint>
-    <link name="base_link">
-        <visual>
-            <geometry>
-                <box size="${base_length} ${base_width} ${base_height}"/>
-            </geometry>
-            <material name="Blue">
-                <color rgba="0 0 1.0 1.0"/>
-            </material>
-        </visual>
-        <collision>
-            <geometry>
-                <box size="${base_length} ${base_width} ${base_height}"/>
-            </geometry>
-        </collision>
-        <xacro:box_inertia m="15" w="${base_width}" d="${base_length}" h="${base_height}"/>
-    </link>
-    <gazebo reference="base_link">
-        <material>Gazebo/Blue</material>
-    </gazebo>
-    <!-- Wheels -->
-    <xacro:macro name="wheel" params="prefix x_reflect y_reflect">
-        <link name="${prefix}_link">
-            <visual>
-                <origin xyz="0 0 0" rpy="${pi/2} 0 0"/>
-                <geometry>
-                    <cylinder radius="${wheel_radius}" length="${wheel_width}"/>
-                </geometry>
-                <material name="Gray">
-                    <color rgba="0.5 0.5 0.5 1.0"/>
-                </material>
-            </visual>
-            <collision>
-                <origin xyz="0 0 0" rpy="${pi/2} 0 0"/>
-                <geometry>
-                    <cylinder radius="${wheel_radius}" length="${wheel_width}"/>
-                </geometry>
-            </collision>
-            <xacro:cylinder_inertia m="0.5" r="${wheel_radius}" h="${wheel_width}"/>
-        </link>
-        <joint name="${prefix}_joint" type="continuous">
-            <parent link="base_link"/>
-            <child link="${prefix}_link"/>
-            <origin xyz="${x_reflect*wheel_xoff} ${y_reflect*(base_width/2+wheel_ygap)} ${-wheel_zoff}" rpy="0 0 0"/>
-            <axis xyz="0 1 0"/>
-        </joint>
-    </xacro:macro>
-    <xacro:wheel prefix="drivewhl_l" x_reflect="-1" y_reflect="1"/>
-    <xacro:wheel prefix="drivewhl_r" x_reflect="-1" y_reflect="-1"/>
-    <!-- Caster Wheel -->
-    <link name="front_caster">
-        <visual>
-            <geometry>
-                <sphere radius="${(wheel_radius+wheel_zoff-(base_height/2))}"/>
-            </geometry>
-            <material name="Cyan">
-                <color rgba="0 1.0 1.0 1.0"/>
-            </material>
-        </visual>
-        <collision>
-            <origin xyz="0 0 0" rpy="0 0 0"/>
-            <geometry>
-                <sphere radius="${(wheel_radius+wheel_zoff-(base_height/2))}"/>
-            </geometry>
-        </collision>
-        <xacro:sphere_inertia m="0.5" r="${(wheel_radius+wheel_zoff-(base_height/2))}"/>
-    </link>
-    <joint name="caster_joint" type="fixed">
-        <parent link="base_link"/>
-        <child link="front_caster"/>
-        <origin xyz="${caster_xoff} 0.0 ${-(base_height/2)}" rpy="0 0 0"/>
-    </joint>
-    <!-- Lidar Sensor -->
-    <link name="lidar_link">
-        <visual>
-            <geometry>
-                <cylinder radius="0.05" length="0.04"/>
-            </geometry>
-            <material name="Black">
-                <color rgba="0 0 0 1"/>
-            </material>
-        </visual>
-        <collision>
-            <geometry>
-                <cylinder radius="0.05" length="0.04"/>
-            </geometry>
-        </collision>
-        <xacro:cylinder_inertia m="0.1" r="0.05" h="0.04"/>
-    </link>
-    <joint name="lidar_joint" type="fixed">
-        <parent link="base_link"/>
-        <child link="lidar_link"/>
-        <origin xyz="0.15 0 0.12" rpy="0 0 0"/>
-    </joint>
-    <!-- Gazebo Plugins -->
-    <gazebo reference="drivewhl_l_link">
-        <mu1>100000.0</mu1>
-        <mu2>100000.0</mu2>
-        <kp>1000000.0</kp>
-        <kd>1.0</kd>
-        <minDepth>0.001</minDepth>
-    </gazebo>
-    <gazebo reference="drivewhl_r_link">
-        <mu1>100000.0</mu1>
-        <mu2>100000.0</mu2>
-        <kp>1000000.0</kp>
-        <kd>1.0</kd>
-        <minDepth>0.001</minDepth>
-    </gazebo>
-    <gazebo>
-        <plugin name='diff_drive' filename='libgazebo_ros_diff_drive.so'>
-            <ros>
-                <!-- Namespace irrelevant for global robot -->
-            </ros>
-            <left_joint>drivewhl_l_joint</left_joint>
-            <right_joint>drivewhl_r_joint</right_joint>
-            <wheel_separation>0.45</wheel_separation>
-            <wheel_diameter>0.2</wheel_diameter>
-            <max_wheel_torque>20</max_wheel_torque>
-            <max_wheel_acceleration>1.0</max_wheel_acceleration>
-            <command_topic>cmd_vel</command_topic>
-            <publish_odom>true</publish_odom>
-            <publish_odom_tf>true</publish_odom_tf>
-            <publish_wheel_tf>true</publish_wheel_tf>
-            <odometry_frame>odom</odometry_frame>
-            <robot_base_frame>base_footprint</robot_base_frame>
-        </plugin>
-    </gazebo>
-    <gazebo reference="lidar_link">
-        <sensor name="lidar" type="ray">
-            <always_on>true</always_on>
-            <!-- Disable visualization to reduce lag -->
-            <visualize>false</visualize>
-            <update_rate>1</update_rate>
-            <ray>
-                <scan>
-                    <horizontal>
-                        <!-- Reduce samples from 360 to 120 -->
-                        <samples>120</samples>
-                        <resolution>1.000000</resolution>
-                        <min_angle>0.000000</min_angle>
-                        <max_angle>6.280000</max_angle>
-                    </horizontal>
-                </scan>
-                <range>
-                    <min>0.120000</min>
-                    <max>3.5</max>
-                    <resolution>0.015000</resolution>
-                </range>
-                <noise>
-                    <type>gaussian</type>
-                    <mean>0.0</mean>
-                    <stddev>0.01</stddev>
-                </noise>
-            </ray>
-            <plugin name="scan" filename="libgazebo_ros_ray_sensor.so">
-                <ros>
-                    <remapping>~/out:=scan</remapping>
-                </ros>
-                <output_type>sensor_msgs/LaserScan</output_type>
-                <frame_name>lidar_link</frame_name>
-            </plugin>
-        </sensor>
-    </gazebo>
+    <!-- Modular URDF components -->
+    <xacro:include filename="common_properties.xacro" />
+    <xacro:include filename="mobile_base.xacro" />
+    <xacro:include filename="mobile_base_gazebo.xacro" />
+    <xacro:include filename="arm.xacro" />
+    <xacro:include filename="sensors.xacro" />
 </robot>
